Commit message: Add camera in simulation

File: smb_description/urdf/sensor_plugins/smb_mono.gazebo.xacro (robot description, xacro)
@@ -10,5 +10,6 @@
     <xacro:property name="mono_update_rate"		value="30"/>
     <xacro:property name="mono_link"  			value="mono_link"/>
-    <xacro:property name="mono_topic" 			value="/mono/cam0/image_raw"/>
+    <xacro:property name="mono_topic" 			value="/versavis/cam0/slow/image_raw"/>
+    <xacro:property name="mono_topic_info" 			value="/versavis/cam0/slow/camera_info"/>
     <link name="${mono_link}">
       <inertial>
@@ -73,5 +74,5 @@
           <cameraName>mono_cam</cameraName>
           <imageTopicName>${mono_topic}</imageTopicName>
-          <cameraInfoTopicName>camera_info</cameraInfoTopicName>
+          <cameraInfoTopicName>${mono_topic_info}</cameraInfoTopicName>
           <frameName>${mono_link}</frameName>
           <hackBaseline>0.07</hackBaseline>

File: smb_description/urdf/smb.urdf.xacro (robot description, xacro)
@@ -163,5 +163,6 @@
         <xacro:IMU base_link="${base_link_name}" simulation="${simulation}"/>
         <!-- <xacro:GPS base_link="${base_link_name}" simulation="${simulation}"/> -->
-        <!-- <xacro:mono_cam base_link="${base_link_name}" simulation="${simulation}"/>
+        <xacro:mono_cam base_link="${base_link_name}" simulation="${simulation}"/>
+        <!--
         <xacro:blackfly_cam id="0" base_link="${base_link_name}" simulation="${simulation}">
             <origin xyz="0.29082 0.04458 ${0.0955 + chassisHeight/2.0}" rpy="0 0 0" />
